File: hardware/button-grid/button_grid.kicad_pcb (KiCad board)
At the start: 2 copper layers, 319.8 x 179.4 mm, 386 parts, among them J1 COL+PWR, J2 ROWS, SW1 PG1350, SW10 PG1350, SW100 PG1350, SW101 PG1350, SW102 PG1350, SW103 PG1350, SW104 PG1350, SW105 PG1350, SW106 PG1350, SW107 PG1350, SW108 PG1350, SW109 PG1350, SW11 PG1350, SW110 PG1350, SW111 PG1350, SW112 PG1350, SW113 PG1350, SW114 PG1350, SW115 PG1350, SW116 PG1350, SW117 PG1350, SW118 PG1350, SW119 PG1350, SW12 PG1350, SW120 PG1350, SW121 PG1350, SW122 PG1350, SW123 PG1350, SW124 PG1350, SW125 PG1350, SW126 PG1350, SW127 PG1350, SW128 PG1350, SW13 PG1350, SW14 PG1350, SW15 PG1350, SW16 PG1350, SW17 PG1350, SW18 PG1350, SW19 PG1350, SW2 PG1350, SW20 PG1350, SW21 PG1350, SW22 PG1350, SW23 PG1350, SW24 PG1350, SW25 PG1350, SW26 PG1350, SW27 PG1350, SW28 PG1350, SW29 PG1350, SW3 PG1350, SW30 PG1350, SW31 PG1350, SW32 PG1350, SW33 PG1350, SW34 PG1350, SW35 PG1350, SW36 PG1350, SW37 PG1350, SW38 PG1350, SW39 PG1350, SW4 PG1350, SW40 PG1350, SW41 PG1350, SW42 PG1350, SW43 PG1350, SW44 PG1350, SW45 PG1350, SW46 PG1350, SW47 PG1350, SW48 PG1350, SW49 PG1350, SW5 PG1350, SW50 PG1350, SW51 PG1350, SW52 PG1350, SW53 PG1350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

Commit message: Add full trace routing to button grid PCB
Routing (1117 traces, 639 vias):
- F.Cu column buses with dogleg around center posts
- F.Cu switch-to-diode traces
- B.Cu row buses with vias at diode cathodes
- B.Cu LED data chain (snaking, intra-row channel + inter-row margin routing)
- B.Cu LED VCC bus (0.5mm power traces at cy-4.5mm per row)
- LED GND vias to B.Cu ground fill
Connector fan-out left for manual routing in KiCad.

https://claude.ai/code/session_01ExJ7gFQfT848CsR2EsnjBp
Routing:
- net VCC: track 0.00 -> 2439.6 mm, vias 0 -> 128
- net ROW7: track 0.00 -> 285.8 mm, vias 0 -> 16
- net ROW6: track 0.00 -> 285.8 mm, vias 0 -> 16
- net ROW5: track 0.00 -> 285.8 mm, vias 0 -> 16
- net ROW4: track 0.00 -> 285.8 mm, vias 0 -> 16
- net ROW3: track 0.00 -> 285.8 mm, vias 0 -> 16
- net ROW2: track 0.00 -> 285.8 mm, vias 0 -> 16
- net ROW1: track 0.00 -> 285.8 mm, vias 0 -> 16
- net ROW0: track 0.00 -> 285.8 mm, vias 0 -> 16
- net COL9: track 0.00 -> 153.4 mm
- net COL8: track 0.00 -> 153.4 mm
- net COL7: track 0.00 -> 153.4 mm
- net COL6: track 0.00 -> 153.4 mm
- net COL5: track 0.00 -> 153.4 mm
- net COL4: track 0.00 -> 153.4 mm
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