File: hardware/button-grid/button_grid.kicad_pcb (KiCad board)
At the start: 2 copper layers, 319.8 x 179.4 mm, 386 parts, among them J1 COL+PWR, J2 ROWS, SW1 PG1350, SW10 PG1350, SW100 PG1350, SW101 PG1350, SW102 PG1350, SW103 PG1350, SW104 PG1350, SW105 PG1350, SW106 PG1350, SW107 PG1350, SW108 PG1350, SW109 PG1350, SW11 PG1350, SW110 PG1350, SW111 PG1350, SW112 PG1350, SW113 PG1350, SW114 PG1350, SW115 PG1350, SW116 PG1350, SW117 PG1350, SW118 PG1350, SW119 PG1350, SW12 PG1350, SW120 PG1350, SW121 PG1350, SW122 PG1350, SW123 PG1350, SW124 PG1350, SW125 PG1350, SW126 PG1350, SW127 PG1350, SW128 PG1350, SW13 PG1350, SW14 PG1350, SW15 PG1350, SW16 PG1350, SW17 PG1350, SW18 PG1350, SW19 PG1350, SW2 PG1350, SW20 PG1350, SW21 PG1350, SW22 PG1350, SW23 PG1350, SW24 PG1350, SW25 PG1350, SW26 PG1350, SW27 PG1350, SW28 PG1350, SW29 PG1350, SW3 PG1350, SW30 PG1350, SW31 PG1350, SW32 PG1350, SW33 PG1350, SW34 PG1350, SW35 PG1350, SW36 PG1350, SW37 PG1350, SW38 PG1350, SW39 PG1350, SW4 PG1350, SW40 PG1350, SW41 PG1350, SW42 PG1350, SW43 PG1350, SW44 PG1350, SW45 PG1350, SW46 PG1350, SW47 PG1350, SW48 PG1350, SW49 PG1350, SW5 PG1350, SW50 PG1350, SW51 PG1350, SW52 PG1350, SW53 PG1350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

Commit message: Tracing
Parts:
- moved J1 335.0 mm to (320.8, 32.3)
- moved J2 297.2 mm to (320.8, 9.50)
Routing:
- net LED_DIN: track 0.00 -> 545.4 mm
- net COL0: track 153.4 -> 505.8 mm
- net COL1: track 153.4 -> 488.3 mm
- net COL2: track 153.4 -> 470.8 mm
- net COL3: track 153.4 -> 453.2 mm
- net COL4: track 153.4 -> 435.7 mm
- net COL5: track 153.4 -> 418.2 mm
- net COL6: track 153.4 -> 400.7 mm
- net COL7: track 153.4 -> 383.2 mm
- net COL8: track 153.4 -> 365.7 mm
- net COL9: track 153.4 -> 348.2 mm
- net COL10: track 153.4 -> 330.7 mm
- net COL11: track 153.4 -> 313.2 mm
- net ROW7: track 285.8 -> 429.1 mm
- net COL12: track 153.4 -> 295.7 mm
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Other:
- board size 319.8 x 179.4 mm -> 322.8 x 167.4 mm

Commit message: Grid pcb scripts
Parts:
- removed J1: COL+PWR, Arp3:PinHeader_1x20_P2.54mm
- removed J2: ROWS, Arp3:PinHeader_1x08_P2.54mm
- added C1: 100nF, Arp3:C_0603, F.Cu at (339.6, 68.4)
- added C2: 100nF, Arp3:C_0603, F.Cu at (339.6, 150.4)
- added C3: 100nF, Arp3:C_0603, F.Cu at (15.5, 168.9)
- added C4: 100nF, Arp3:C_0603, F.Cu at (15.5, 170.9)
- added C5: 100nF, Arp3:C_0603, F.Cu at (263.2, 178.4)
- added C6: 100nF, Arp3:C_0603, F.Cu at (263.2, 180.4)
- added R1: 4.7k, Arp3:C_0603, F.Cu at (339.2, 63.4)
- added R2: 4.7k, Arp3:C_0603, F.Cu at (339.2, 65.4)
- added SW_CMD: , Arp3:Kailh_Choc_V1, F.Cu at (87.7, 163.9)
- added SW_CTRL: , Arp3:Kailh_Choc_V1, F.Cu at (49.6, 163.9)
- added SW_OPT: , Arp3:Kailh_Choc_V1, F.Cu at (68.7, 163.9)
- added SW_SHIFT: , Arp3:Kailh_Choc_V1, F.Cu at (30.6, 163.9)
- added SW_SPACE: , Arp3:Kailh_Choc_V1, F.Cu at (135.3, 163.9)
- added U1: MCP23017, Arp3:MCP23017_QFN28, F.Cu at (334.6, 68.4)
- added U2: MCP23017, Arp3:MCP23017_QFN28, F.Cu at (334.6, 150.4)
- added U3: Teensy 4.1, Arp3:Teensy41, F.Cu at (339.2, 2.00)
- added U3: MPR121, Arp3:MPR121_QFN20, F.Cu at (11.5, 168.9)
- added U4: MPR121, Arp3:MPR121_QFN20, F.Cu at (259.2, 178.4)
- moved D10 14.6 mm to (207.0, 18.5)
- moved D101 14.6 mm to (111.8, 132.8)
- moved D103 14.6 mm to (149.9, 132.8)
- moved D104 14.6 mm to (168.9, 132.8)
- moved D106 14.6 mm to (207.0, 132.8)
- moved D108 14.6 mm to (245.1, 132.8)
- moved D109 14.6 mm to (264.2, 132.8)
- moved D110 14.6 mm to (283.2, 132.8)
- moved D112 14.6 mm to (321.3, 132.8)
- moved D117 14.6 mm to (111.8, 151.9)
- moved D119 14.6 mm to (149.9, 151.9)
- moved D12 14.6 mm to (245.1, 18.5)
- moved D120 14.6 mm to (168.9, 151.9)
- moved D122 14.6 mm to (207.0, 151.9)
- moved D124 14.6 mm to (245.1, 151.9)
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Routing:
- net LED_DIN: track 545.4 -> 0.00 mm
- net COL0: track 505.8 -> 741.9 mm, vias 0 -> 4
- net COL1: track 488.3 -> 703.8 mm, vias 0 -> 4
- net COL2: track 470.8 -> 665.6 mm, vias 0 -> 4
- net COL3: track 453.2 -> 627.5 mm, vias 0 -> 4
- net COL4: track 435.7 -> 589.5 mm, vias 0 -> 4
- net ROW7: track 429.1 -> 285.8 mm
- net COL5: track 418.2 -> 551.4 mm, vias 0 -> 4
- net ROW6: track 412.6 -> 285.8 mm
- net COL6: track 400.7 -> 513.2 mm, vias 0 -> 4
- net ROW5: track 396.1 -> 285.8 mm
- net ROW4: track 379.6 -> 285.8 mm
- net COL7: track 383.2 -> 475.1 mm, vias 0 -> 4
- net ROW3: track 363.1 -> 285.8 mm
- net COL15: track 243.1 -> 170.4 mm, vias 0 -> 4
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- added copper zone on F.Cu, net HSLIDER0
- added copper zone on F.Cu, net HSLIDER1
- added copper zone on F.Cu, net HSLIDER2
- added copper zone on F.Cu, net HSLIDER3
- added copper zone on F.Cu, net HSLIDER4
- added copper zone on F.Cu, net HSLIDER5
- added copper zone on F.Cu, net HSLIDER6
- added copper zone on F.Cu, net HSLIDER7
- added copper zone on F.Cu, net VSLIDER0
- added copper zone on F.Cu, net VSLIDER1
- added copper zone on F.Cu, net VSLIDER2
- added copper zone on F.Cu, net VSLIDER3
- added copper zone on F.Cu, net VSLIDER4
- added copper zone on F.Cu, net VSLIDER5
- added copper zone on F.Cu, net VSLIDER6
- added copper zone on F.Cu, net VSLIDER7
Other:
- board size 322.8 x 167.4 mm -> 349.9 x 175.4 mm

Commit message: Better components
Parts:
- added C7: 10uF, Arp3:C_0603, F.Cu at (381.9, 7.00)
- added J2: TFT 2.4in, Arp3:ILI9341_2.4inch, F.Cu at (328.9, 23.5)
- added J3: USB-C, Arp3:USB_C_Mid_Mount, F.Cu at (381.9, 0.00)
- added R3: 5.1k, Arp3:R_0603, F.Cu at (379.9, 5.00)
- added R4: 5.1k, Arp3:R_0603, F.Cu at (383.9, 5.00)
- R1, R2: footprint Arp3:C_0603 -> Arp3:R_0603
- moved R1 21.1 mm to (360.4, 63.4)
- moved R2 21.1 mm to (360.4, 65.4)
- moved U3 21.1 mm to (360.4, 2.00)
- moved C1 5.76 mm to (345.4, 68.4)
- moved C2 5.76 mm to (345.4, 150.4)
- moved U1 5.76 mm to (340.4, 68.4)
- moved U2 5.76 mm to (340.4, 150.4)
Other:
- board size 349.9 x 175.4 mm -> 393.9 x 175.4 mm

Commit message: Improve pcb
Parts:
- moved D1 13.5 mm to (22.1, 18.5)
- moved D113 13.5 mm to (22.1, 151.9)
- moved D17 13.5 mm to (22.1, 37.6)
- moved D33 13.5 mm to (22.1, 56.6)
- moved D49 13.5 mm to (22.1, 75.7)
- moved D65 13.5 mm to (22.1, 94.7)
- moved D81 13.5 mm to (22.1, 113.8)
- moved D97 13.5 mm to (22.1, 132.8)
- moved D10 13.5 mm to (193.5, 18.5)
- moved D100 13.5 mm to (79.2, 132.8)
- moved D101 13.5 mm to (98.3, 132.8)
- moved D103 13.5 mm to (136.4, 132.8)
- moved D104 13.5 mm to (155.4, 132.8)
- moved D105 13.5 mm to (174.5, 132.8)
- moved D106 13.5 mm to (193.5, 132.8)
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Routing:
- net VCC: track 2439.6 -> 0.00 mm
- net COL7: track 475.1 -> 447.7 mm
- net COL6: track 513.2 -> 485.8 mm
- net COL5: track 551.4 -> 523.9 mm
- net COL4: track 589.5 -> 562.0 mm
- net COL13: track 246.5 -> 219.1 mm
- net COL12: track 284.6 -> 257.2 mm
- net COL11: track 322.8 -> 295.3 mm
- net COL1: track 703.8 -> 676.3 mm
- net COL0: track 741.9 -> 714.4 mm
- net COL9: track 398.9 -> 371.5 mm
- net COL8: track 437.1 -> 409.6 mm
- net COL3: track 627.5 -> 600.1 mm
- net COL2: track 665.6 -> 638.2 mm
- net COL14: track 208.5 -> 181.0 mm
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- added copper zone on B.Cu, net VCC
