File: hardware/button_grid.kicad_pcb (KiCad board)
At the start: 2 copper layers, 393.9 x 175.4 mm, 407 parts, among them J2 TFT 2.4in, J3 USB-C, SW1 PG1350, SW10 PG1350, SW100 PG1350, SW101 PG1350, SW102 PG1350, SW103 PG1350, SW104 PG1350, SW105 PG1350, SW106 PG1350, SW107 PG1350, SW108 PG1350, SW109 PG1350, SW11 PG1350, SW110 PG1350, SW111 PG1350, SW112 PG1350, SW113 PG1350, SW114 PG1350, SW115 PG1350, SW116 PG1350, SW117 PG1350, SW118 PG1350, SW119 PG1350, SW12 PG1350, SW120 PG1350, SW121 PG1350, SW122 PG1350, SW123 PG1350, SW124 PG1350, SW125 PG1350, SW126 PG1350, SW127 PG1350, SW128 PG1350, SW13 PG1350, SW14 PG1350, SW15 PG1350, SW16 PG1350, SW17 PG1350, SW18 PG1350, SW19 PG1350, SW2 PG1350, SW20 PG1350, SW21 PG1350, SW22 PG1350, SW23 PG1350, SW24 PG1350, SW25 PG1350, SW26 PG1350, SW27 PG1350, SW28 PG1350, SW29 PG1350, SW3 PG1350, SW30 PG1350, SW31 PG1350, SW32 PG1350, SW33 PG1350, SW34 PG1350, SW35 PG1350, SW36 PG1350, SW37 PG1350, SW38 PG1350, SW39 PG1350, SW4 PG1350, SW40 PG1350, SW41 PG1350, SW42 PG1350, SW43 PG1350, SW44 PG1350, SW45 PG1350, SW46 PG1350, SW47 PG1350, SW48 PG1350, SW49 PG1350, SW5 PG1350, SW50 PG1350, SW51 PG1350, SW52 PG1350, SW53 PG1350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

Commit message: Trace bottom buttons
Parts:
- removed SW_CMD, SW_CTRL, SW_OPT, SW_SHIFT, SW_SPACE: , Arp3:Kailh_Choc_V1
- added D_R9_0: , Arp3:D_SOD-323, F.Cu at (3.02, 170.9)
- added D_R9_1: , Arp3:D_SOD-323, F.Cu at (22.1, 170.9)
- added D_R9_2: , Arp3:D_SOD-323, F.Cu at (41.1, 170.9)
- added D_R9_3: , Arp3:D_SOD-323, F.Cu at (60.2, 170.9)
- added D_R9_4: , Arp3:D_SOD-323, F.Cu at (79.2, 170.9)
- added D_R9_5: , Arp3:D_SOD-323, F.Cu at (98.3, 170.9)
- added D_R9_6: , Arp3:D_SOD-323, F.Cu at (117.3, 170.9)
- added D_R9_7: , Arp3:D_SOD-323, F.Cu at (136.4, 170.9)
- added D_R9_8: , Arp3:D_SOD-323, F.Cu at (155.4, 170.9)
- added SW_R9_0: , Arp3:Kailh_Choc_V1, F.Cu at (11.5, 163.9)
- added SW_R9_1: , Arp3:Kailh_Choc_V1, F.Cu at (30.6, 163.9)
- added SW_R9_2: , Arp3:Kailh_Choc_V1, F.Cu at (49.6, 163.9)
- added SW_R9_3: , Arp3:Kailh_Choc_V1, F.Cu at (68.7, 163.9)
- added SW_R9_4: , Arp3:Kailh_Choc_V1, F.Cu at (87.7, 163.9)
- added SW_R9_5: , Arp3:Kailh_Choc_V1, F.Cu at (106.8, 163.9)
- added SW_R9_6: , Arp3:Kailh_Choc_V1, F.Cu at (125.8, 163.9)
- added SW_R9_7: , Arp3:Kailh_Choc_V1, F.Cu at (144.9, 163.9)
- added SW_R9_8: , Arp3:Kailh_Choc_V1, F.Cu at (163.9, 163.9)
- C3, C4, C5, C6, U3, U4: moved to B.Cu
- moved C3 81.2 mm to (15.5, 87.7)
- moved C4 81.2 mm to (15.5, 89.7)
- moved U3 81.2 mm to (11.5, 87.7)
- moved C5 14.5 mm to (263.2, 163.9)
- moved C6 14.5 mm to (263.2, 165.9)
- moved U4 14.5 mm to (259.2, 163.9)
Routing:
- net ROW8: track 0.00 -> 152.4 mm, vias 0 -> 9
- net COL7: track 447.7 -> 502.9 mm
- net COL6: track 485.8 -> 541.0 mm
- net COL5: track 523.9 -> 579.1 mm
- net COL4: track 562.0 -> 617.2 mm
- net COL3: track 600.1 -> 655.3 mm
- net COL2: track 638.2 -> 693.4 mm
- net COL1: track 676.3 -> 731.5 mm
- net COL0: track 714.4 -> 769.6 mm
- net COL11: track 295.3 -> 329.1 mm
- net COL10: track 333.4 -> 367.2 mm
- net COL14: track 181.0 -> 214.8 mm
- net COL9: track 371.5 -> 405.3 mm
- net COL8: track 409.6 -> 443.4 mm
- net COL13: track 219.1 -> 252.9 mm
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
Commit message: PCB tweaks + bom generator
Parts:
- removed C3: 100nF, Arp3:C_0603
- removed the C5 at (263.2, 163.9)
- added C5: 100nF, Arp3:C_0603, B.Cu at (15.5, 146.9)
- added C5: 100nF, Arp3:C_0603, B.Cu at (320.3, 163.9)
- added C8: 100uF, Arp3:C_0603, F.Cu at (378.9, 13.0)
- added C9: 10uF, Arp3:C_0603, F.Cu at (384.9, 15.0)
- added D_TVS3_0: PRTR5V0U2X, Arp3:PRTR5V0U2X_SOT-143B, B.Cu at (7.53, 141.9)
- added D_TVS3_1: PRTR5V0U2X, Arp3:PRTR5V0U2X_SOT-143B, B.Cu at (7.53, 144.4)
- added D_TVS3_2: PRTR5V0U2X, Arp3:PRTR5V0U2X_SOT-143B, B.Cu at (7.53, 146.9)
- added D_TVS3_3: PRTR5V0U2X, Arp3:PRTR5V0U2X_SOT-143B, B.Cu at (7.53, 149.4)
- added D_TVS4_0: PRTR5V0U2X, Arp3:PRTR5V0U2X_SOT-143B, B.Cu at (312.3, 160.9)
- added D_TVS4_1: PRTR5V0U2X, Arp3:PRTR5V0U2X_SOT-143B, B.Cu at (312.3, 163.4)
- added D_TVS4_2: PRTR5V0U2X, Arp3:PRTR5V0U2X_SOT-143B, B.Cu at (312.3, 165.9)
- added D_TVS4_3: PRTR5V0U2X, Arp3:PRTR5V0U2X_SOT-143B, B.Cu at (312.3, 168.4)
- added F1: 2A PTC, Arp3:R_0603, F.Cu at (381.9, 10.0)
- added FB1: 600R@100MHz, Arp3:R_0603, F.Cu at (384.9, 13.0)
- added R5: 0R, Arp3:R_0603, F.Cu at (381.9, 13.0)
- moved U1 62.2 mm to (330.9, 7.00), turned to 90 degrees
- moved C1 58.3 mm to (330.9, 12.0)
- moved U3 57.2 mm to (11.5, 144.9)
- moved C6 57.1 mm to (320.3, 165.9)
- moved U4 57.1 mm to (316.3, 163.9)
- moved C4 55.2 mm to (15.5, 144.9)
- moved C2 15.7 mm to (330.9, 144.4)
- moved U2 9.58 mm to (330.9, 149.4), turned to 90 degrees
Connections:
- LED1 pad 1: VCC -> LED_VCC
- LED10 pad 1: VCC -> LED_VCC
- LED100 pad 1: VCC -> LED_VCC
- LED101 pad 1: VCC -> LED_VCC
- LED102 pad 1: VCC -> LED_VCC
- LED103 pad 1: VCC -> LED_VCC
- LED104 pad 1: VCC -> LED_VCC
- LED105 pad 1: VCC -> LED_VCC
- LED106 pad 1: VCC -> LED_VCC
- LED107 pad 1: VCC -> LED_VCC
- LED108 pad 1: VCC -> LED_VCC
- LED109 pad 1: VCC -> LED_VCC
- LED11 pad 1: VCC -> LED_VCC
- LED110 pad 1: VCC -> LED_VCC
- LED111 pad 1: VCC -> LED_VCC
- LED112 pad 1: VCC -> LED_VCC
- LED113 pad 1: VCC -> LED_VCC
- LED114 pad 1: VCC -> LED_VCC
- LED115 pad 1: VCC -> LED_VCC
- LED116 pad 1: VCC -> LED_VCC
- LED117 pad 1: VCC -> LED_VCC
- LED118 pad 1: VCC -> LED_VCC
- LED119 pad 1: VCC -> LED_VCC
- LED12 pad 1: VCC -> LED_VCC
- LED120 pad 1: VCC -> LED_VCC
- LED121 pad 1: VCC -> LED_VCC
- LED122 pad 1: VCC -> LED_VCC
- LED123 pad 1: VCC -> LED_VCC
- LED124 pad 1: VCC -> LED_VCC
- LED125 pad 1: VCC -> LED_VCC
- LED126 pad 1: VCC -> LED_VCC
- LED127 pad 1: VCC -> LED_VCC
- LED128 pad 1: VCC -> LED_VCC
- LED13 pad 1: VCC -> LED_VCC
- LED14 pad 1: VCC -> LED_VCC
- LED15 pad 1: VCC -> LED_VCC
- LED16 pad 1: VCC -> LED_VCC
- LED17 pad 1: VCC -> LED_VCC
- LED18 pad 1: VCC -> LED_VCC
- LED19 pad 1: VCC -> LED_VCC
- LED2 pad 1: VCC -> LED_VCC
- LED20 pad 1: VCC -> LED_VCC
- LED21 pad 1: VCC -> LED_VCC
- LED22 pad 1: VCC -> LED_VCC
- LED23 pad 1: VCC -> LED_VCC
- LED24 pad 1: VCC -> LED_VCC
- LED25 pad 1: VCC -> LED_VCC
- LED26 pad 1: VCC -> LED_VCC
- LED27 pad 1: VCC -> LED_VCC
- LED28 pad 1: VCC -> LED_VCC
- LED29 pad 1: VCC -> LED_VCC
- LED3 pad 1: VCC -> LED_VCC
- LED30 pad 1: VCC -> LED_VCC
- LED31 pad 1: VCC -> LED_VCC
- LED32 pad 1: VCC -> LED_VCC
- LED33 pad 1: VCC -> LED_VCC
- LED34 pad 1: VCC -> LED_VCC
- LED35 pad 1: VCC -> LED_VCC
- LED36 pad 1: VCC -> LED_VCC
- LED37 pad 1: VCC -> LED_VCC
- LED38 pad 1: VCC -> LED_VCC
- LED39 pad 1: VCC -> LED_VCC
- LED4 pad 1: VCC -> LED_VCC
- LED40 pad 1: VCC -> LED_VCC
- LED41 pad 1: VCC -> LED_VCC
- LED42 pad 1: VCC -> LED_VCC
- LED43 pad 1: VCC -> LED_VCC
- LED44 pad 1: VCC -> LED_VCC
- LED45 pad 1: VCC -> LED_VCC
- LED46 pad 1: VCC -> LED_VCC
- LED47 pad 1: VCC -> LED_VCC
- LED48 pad 1: VCC -> LED_VCC
- LED49 pad 1: VCC -> LED_VCC
- LED5 pad 1: VCC -> LED_VCC
- LED50 pad 1: VCC -> LED_VCC
- LED51 pad 1: VCC -> LED_VCC
- LED52 pad 1: VCC -> LED_VCC
- LED53 pad 1: VCC -> LED_VCC
- LED54 pad 1: VCC -> LED_VCC
- LED55 pad 1: VCC -> LED_VCC
- LED56 pad 1: VCC -> LED_VCC
- LED57 pad 1: VCC -> LED_VCC
- LED58 pad 1: VCC -> LED_VCC
- LED59 pad 1: VCC -> LED_VCC
- LED6 pad 1: VCC -> LED_VCC
- LED60 pad 1: VCC -> LED_VCC
- LED61 pad 1: VCC -> LED_VCC
- LED62 pad 1: VCC -> LED_VCC
- LED63 pad 1: VCC -> LED_VCC
- LED64 pad 1: VCC -> LED_VCC
- LED65 pad 1: VCC -> LED_VCC
- LED66 pad 1: VCC -> LED_VCC
- LED67 pad 1: VCC -> LED_VCC
- LED68 pad 1: VCC -> LED_VCC
- LED69 pad 1: VCC -> LED_VCC
- LED7 pad 1: VCC -> LED_VCC
- LED70 pad 1: VCC -> LED_VCC
- LED71 pad 1: VCC -> LED_VCC
- LED72 pad 1: VCC -> LED_VCC
- LED73 pad 1: VCC -> LED_VCC
- LED74 pad 1: VCC -> LED_VCC
- LED75 pad 1: VCC -> LED_VCC
- LED76 pad 1: VCC -> LED_VCC
- LED77 pad 1: VCC -> LED_VCC
- LED78 pad 1: VCC -> LED_VCC
- LED79 pad 1: VCC -> LED_VCC
- LED8 pad 1: VCC -> LED_VCC
- LED80 pad 1: VCC -> LED_VCC
- LED81 pad 1: VCC -> LED_VCC
- LED82 pad 1: VCC -> LED_VCC
- LED83 pad 1: VCC -> LED_VCC
- LED84 pad 1: VCC -> LED_VCC
- LED85 pad 1: VCC -> LED_VCC
- LED86 pad 1: VCC -> LED_VCC
- LED87 pad 1: VCC -> LED_VCC
- LED88 pad 1: VCC -> LED_VCC
- LED89 pad 1: VCC -> LED_VCC
- LED9 pad 1: VCC -> LED_VCC
- LED90 pad 1: VCC -> LED_VCC
- LED91 pad 1: VCC -> LED_VCC
- LED92 pad 1: VCC -> LED_VCC
- LED93 pad 1: VCC -> LED_VCC
- LED94 pad 1: VCC -> LED_VCC
- LED95 pad 1: VCC -> LED_VCC
- LED96 pad 1: VCC -> LED_VCC
- LED97 pad 1: VCC -> LED_VCC
- LED98 pad 1: VCC -> LED_VCC
- LED99 pad 1: VCC -> LED_VCC
- SW_R9_0 pad 1: COL_NEG1 -> COL0
- SW_R9_1 pad 1: COL0 -> COL1
- SW_R9_2 pad 1: COL1 -> COL2
- SW_R9_3 pad 1: COL2 -> COL3
- SW_R9_4 pad 1: COL3 -> COL4
- SW_R9_5 pad 1: COL4 -> COL5
- SW_R9_6 pad 1: COL5 -> COL6
- SW_R9_7 pad 1: COL6 -> COL7
- SW_R9_8 pad 1: COL7 -> COL8
- U3 pad 10: VSLIDER1 -> VSLIDER6
- U3 pad 12: VSLIDER2 -> VSLIDER5
- U3 pad 13: VSLIDER3 -> VSLIDER4
- U3 pad 14: VSLIDER4 -> VSLIDER3
- U3 pad 15: VSLIDER5 -> VSLIDER2
- U3 pad 16: VSLIDER6 -> VSLIDER1
- U3 pad 17: VSLIDER7 -> VSLIDER0
- U3 pad 9: VSLIDER0 -> VSLIDER7
Routing:
- net COL0: track 769.6 -> 180.3 mm, vias 4 -> 0
- net COL1: track 731.5 -> 180.3 mm, vias 4 -> 0
- net COL2: track 693.4 -> 180.3 mm, vias 4 -> 0
- net COL3: track 655.3 -> 180.3 mm, vias 4 -> 0
- net COL4: track 617.2 -> 180.3 mm, vias 4 -> 0
- net COL5: track 579.1 -> 180.3 mm, vias 4 -> 0
- net COL6: track 541.0 -> 180.3 mm, vias 4 -> 0
- net COL7: track 502.9 -> 180.3 mm, vias 4 -> 0
- net COL8: track 443.4 -> 180.3 mm, vias 4 -> 2
- net COL9: track 405.3 -> 152.6 mm, vias 4 -> 0
- net COL10: track 367.2 -> 152.6 mm, vias 4 -> 0
- net COL11: track 329.1 -> 152.6 mm, vias 4 -> 0
- net COL12: track 291.0 -> 152.6 mm, vias 4 -> 0
- net COL13: track 252.9 -> 152.6 mm, vias 4 -> 0
- net COL14: track 214.8 -> 152.6 mm, vias 4 -> 0
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- added copper zone on B.Cu, net LED_VCC
- removed copper zone on B.Cu, net VCC

Commit message: Update PCB
Parts:
- removed D1, D10, D100, D101, D102, D103, D104, D105, D106, D107, D108, D109, D11, D110, D111, D112, D113, D114, D115, D116, D117, D118, D119, D12, D120, D121, D122, D123, D124, D125, D126, D127, D128, D13, D14, D15, D16, D17, D18, D19, D2, D20, D21, D22, D23, D24, D25, D26, D27, D28, D29, D3, D30, D31, D32, D33, D34, D35, D36, D37, D38, D39, D4, D40, D41, D42, D43, D44, D45, D46, D47, D48, D49, D5, D50, D51, D52, D53, D54, D55, D56, D57, D58, D59, D6, D60, D61, D62, D63, D64, D65, D66, D67, D68, D69, D7, D70, D71, D72, D73, D74, D75, D76, D77, D78, D79, D8, D80, D81, D82, D83, D84, D85, D86, D87, D88, D89, D9, D90, D91, D92, D93, D94, D95, D96, D97, D98, D99: 1N4148W, Arp3:D_SOD-323
- removed D_R9_0, D_R9_1, D_R9_2, D_R9_3, D_R9_4, D_R9_5, D_R9_6, D_R9_7, D_R9_8: , Arp3:D_SOD-323
- removed LED1, LED10, LED100, LED101, LED102, LED103, LED104, LED105, LED106, LED107, LED108, LED109, LED11, LED110, LED111, LED112, LED113, LED114, LED115, LED116, LED117, LED118, LED119, LED12, LED120, LED121, LED122, LED123, LED124, LED125, LED126, LED127, LED128, LED13, LED14, LED15, LED16, LED17, LED18, LED19, LED2, LED20, LED21, LED22, LED23, LED24, LED25, LED26, LED27, LED28, LED29, LED3, LED30, LED31, LED32, LED33, LED34, LED35, LED36, LED37, LED38, LED39, LED4, LED40, LED41, LED42, LED43, LED44, LED45, LED46, LED47, LED48, LED49, LED5, LED50, LED51, LED52, LED53, LED54, LED55, LED56, LED57, LED58, LED59, LED6, LED60, LED61, LED62, LED63, LED64, LED65, LED66, LED67, LED68, LED69, LED7, LED70, LED71, LED72, LED73, LED74, LED75, LED76, LED77, LED78, LED79, LED8, LED80, LED81, LED82, LED83, LED84, LED85, LED86, LED87, LED88, LED89, LED9, LED90, LED91, LED92, LED93, LED94, LED95, LED96, LED97, LED98, LED99: SK6812MINI-E, Arp3:SK6812MINI-E
- removed SW1, SW10, SW100, SW101, SW102, SW103, SW104, SW105, SW106, SW107, SW108, SW109, SW11, SW110, SW111, SW112, SW113, SW114, SW115, SW116, SW117, SW118, SW119, SW12, SW120, SW121, SW122, SW123, SW124, SW125, SW126, SW127, SW128, SW13, SW14, SW15, SW16, SW17, SW18, SW19, SW2, SW20, SW21, SW22, SW23, SW24, SW25, SW26, SW27, SW28, SW29, SW3, SW30, SW31, SW32, SW33, SW34, SW35, SW36, SW37, SW38, SW39, SW4, SW40, SW41, SW42, SW43, SW44, SW45, SW46, SW47, SW48, SW49, SW5, SW50, SW51, SW52, SW53, SW54, SW55, SW56, SW57, SW58, SW59, SW6, SW60, SW61, SW62, SW63, SW64, SW65, SW66, SW67, SW68, SW69, SW7, SW70, SW71, SW72, SW73, SW74, SW75, SW76, SW77, SW78, SW79, SW8, SW80, SW81, SW82, SW83, SW84, SW85, SW86, SW87, SW88, SW89, SW9, SW90, SW91, SW92, SW93, SW94, SW95, SW96, SW97, SW98, SW99: PG1350, Arp3:Kailh_Choc_V1
- removed SW_R9_0, SW_R9_1, SW_R9_2, SW_R9_3, SW_R9_4, SW_R9_5, SW_R9_6, SW_R9_7, SW_R9_8: , Arp3:Kailh_Choc_V1
- added D_R01_C01: 1N4148W, Arp3:D_SOD-323, F.Cu at (22.1, 18.5)
- added D_R01_C02: 1N4148W, Arp3:D_SOD-323, F.Cu at (41.1, 18.5)
- added D_R01_C03: 1N4148W, Arp3:D_SOD-323, F.Cu at (60.2, 18.5)
- added D_R01_C04: 1N4148W, Arp3:D_SOD-323, F.Cu at (79.2, 18.5)
- added D_R01_C05: 1N4148W, Arp3:D_SOD-323, F.Cu at (98.3, 18.5)
- added D_R01_C06: 1N4148W, Arp3:D_SOD-323, F.Cu at (117.3, 18.5)
- added D_R01_C07: 1N4148W, Arp3:D_SOD-323, F.Cu at (136.4, 18.5)
- added D_R01_C08: 1N4148W, Arp3:D_SOD-323, F.Cu at (155.4, 18.5)
- added D_R01_C09: 1N4148W, Arp3:D_SOD-323, F.Cu at (174.5, 18.5)
- added D_R01_C10: 1N4148W, Arp3:D_SOD-323, F.Cu at (193.5, 18.5)
- added D_R01_C11: 1N4148W, Arp3:D_SOD-323, F.Cu at (212.6, 18.5)
- added D_R01_C12: 1N4148W, Arp3:D_SOD-323, F.Cu at (231.6, 18.5)
- added D_R01_C13: 1N4148W, Arp3:D_SOD-323, F.Cu at (250.7, 18.5)
- added D_R01_C14: 1N4148W, Arp3:D_SOD-323, F.Cu at (269.7, 18.5)
- added D_R01_C15: 1N4148W, Arp3:D_SOD-323, F.Cu at (288.8, 18.5)
- added D_R01_C16: 1N4148W, Arp3:D_SOD-323, F.Cu at (307.8, 18.5)
- added D_R02_C01: 1N4148W, Arp3:D_SOD-323, F.Cu at (22.1, 37.6)
- added D_R02_C02: 1N4148W, Arp3:D_SOD-323, F.Cu at (41.1, 37.6)
- added D_R02_C03: 1N4148W, Arp3:D_SOD-323, F.Cu at (60.2, 37.6)
- added D_R02_C04: 1N4148W, Arp3:D_SOD-323, F.Cu at (79.2, 37.6)
- added D_R02_C05: 1N4148W, Arp3:D_SOD-323, F.Cu at (98.3, 37.6)
- added D_R02_C06: 1N4148W, Arp3:D_SOD-323, F.Cu at (117.3, 37.6)
- added D_R02_C07: 1N4148W, Arp3:D_SOD-323, F.Cu at (136.4, 37.6)
- added D_R02_C08: 1N4148W, Arp3:D_SOD-323, F.Cu at (155.4, 37.6)
- added D_R02_C09: 1N4148W, Arp3:D_SOD-323, F.Cu at (174.5, 37.6)
- added D_R02_C10: 1N4148W, Arp3:D_SOD-323, F.Cu at (193.5, 37.6)
- added D_R02_C11: 1N4148W, Arp3:D_SOD-323, F.Cu at (212.6, 37.6)
- added D_R02_C12: 1N4148W, Arp3:D_SOD-323, F.Cu at (231.6, 37.6)
- added D_R02_C13: 1N4148W, Arp3:D_SOD-323, F.Cu at (250.7, 37.6)
- added D_R02_C14: 1N4148W, Arp3:D_SOD-323, F.Cu at (269.7, 37.6)
- added D_R02_C15: 1N4148W, Arp3:D_SOD-323, F.Cu at (288.8, 37.6)
- added D_R02_C16: 1N4148W, Arp3:D_SOD-323, F.Cu at (307.8, 37.6)
- added D_R03_C01: 1N4148W, Arp3:D_SOD-323, F.Cu at (22.1, 56.6)
- added D_R03_C02: 1N4148W, Arp3:D_SOD-323, F.Cu at (41.1, 56.6)
- added D_R03_C03: 1N4148W, Arp3:D_SOD-323, F.Cu at (60.2, 56.6)
- added D_R03_C04: 1N4148W, Arp3:D_SOD-323, F.Cu at (79.2, 56.6)
- added D_R03_C05: 1N4148W, Arp3:D_SOD-323, F.Cu at (98.3, 56.6)
- added D_R03_C06: 1N4148W, Arp3:D_SOD-323, F.Cu at (117.3, 56.6)
- added D_R03_C07: 1N4148W, Arp3:D_SOD-323, F.Cu at (136.4, 56.6)
- added D_R03_C08: 1N4148W, Arp3:D_SOD-323, F.Cu at (155.4, 56.6)
- added D_R03_C09: 1N4148W, Arp3:D_SOD-323, F.Cu at (174.5, 56.6)
- added D_R03_C10: 1N4148W, Arp3:D_SOD-323, F.Cu at (193.5, 56.6)
- added D_R03_C11: 1N4148W, Arp3:D_SOD-323, F.Cu at (212.6, 56.6)
- added D_R03_C12: 1N4148W, Arp3:D_SOD-323, F.Cu at (231.6, 56.6)
- added D_R03_C13: 1N4148W, Arp3:D_SOD-323, F.Cu at (250.7, 56.6)
- added D_R03_C14: 1N4148W, Arp3:D_SOD-323, F.Cu at (269.7, 56.6)
- added D_R03_C15: 1N4148W, Arp3:D_SOD-323, F.Cu at (288.8, 56.6)
- added D_R03_C16: 1N4148W, Arp3:D_SOD-323, F.Cu at (307.8, 56.6)
- added D_R04_C01: 1N4148W, Arp3:D_SOD-323, F.Cu at (22.1, 75.7)
- added D_R04_C02: 1N4148W, Arp3:D_SOD-323, F.Cu at (41.1, 75.7)
- added D_R04_C03: 1N4148W, Arp3:D_SOD-323, F.Cu at (60.2, 75.7)
- added D_R04_C04: 1N4148W, Arp3:D_SOD-323, F.Cu at (79.2, 75.7)
- added D_R04_C05: 1N4148W, Arp3:D_SOD-323, F.Cu at (98.3, 75.7)
- added D_R04_C06: 1N4148W, Arp3:D_SOD-323, F.Cu at (117.3, 75.7)
- added D_R04_C07: 1N4148W, Arp3:D_SOD-323, F.Cu at (136.4, 75.7)
- added D_R04_C08: 1N4148W, Arp3:D_SOD-323, F.Cu at (155.4, 75.7)
- added D_R04_C09: 1N4148W, Arp3:D_SOD-323, F.Cu at (174.5, 75.7)
- added D_R04_C10: 1N4148W, Arp3:D_SOD-323, F.Cu at (193.5, 75.7)
- added D_R04_C11: 1N4148W, Arp3:D_SOD-323, F.Cu at (212.6, 75.7)
- added D_R04_C12: 1N4148W, Arp3:D_SOD-323, F.Cu at (231.6, 75.7)
- added D_R04_C13: 1N4148W, Arp3:D_SOD-323, F.Cu at (250.7, 75.7)
- added D_R04_C14: 1N4148W, Arp3:D_SOD-323, F.Cu at (269.7, 75.7)
- added D_R04_C15: 1N4148W, Arp3:D_SOD-323, F.Cu at (288.8, 75.7)
- added D_R04_C16: 1N4148W, Arp3:D_SOD-323, F.Cu at (307.8, 75.7)
- added D_R05_C01: 1N4148W, Arp3:D_SOD-323, F.Cu at (22.1, 94.7)
- added D_R05_C02: 1N4148W, Arp3:D_SOD-323, F.Cu at (41.1, 94.7)
- added D_R05_C03: 1N4148W, Arp3:D_SOD-323, F.Cu at (60.2, 94.7)
- added D_R05_C04: 1N4148W, Arp3:D_SOD-323, F.Cu at (79.2, 94.7)
- added D_R05_C05: 1N4148W, Arp3:D_SOD-323, F.Cu at (98.3, 94.7)
- added D_R05_C06: 1N4148W, Arp3:D_SOD-323, F.Cu at (117.3, 94.7)
- added D_R05_C07: 1N4148W, Arp3:D_SOD-323, F.Cu at (136.4, 94.7)
- added D_R05_C08: 1N4148W, Arp3:D_SOD-323, F.Cu at (155.4, 94.7)
- added D_R05_C09: 1N4148W, Arp3:D_SOD-323, F.Cu at (174.5, 94.7)
- added D_R05_C10: 1N4148W, Arp3:D_SOD-323, F.Cu at (193.5, 94.7)
- added D_R05_C11: 1N4148W, Arp3:D_SOD-323, F.Cu at (212.6, 94.7)
- added D_R05_C12: 1N4148W, Arp3:D_SOD-323, F.Cu at (231.6, 94.7)
- added D_R05_C13: 1N4148W, Arp3:D_SOD-323, F.Cu at (250.7, 94.7)
- added D_R05_C14: 1N4148W, Arp3:D_SOD-323, F.Cu at (269.7, 94.7)
- added D_R05_C15: 1N4148W, Arp3:D_SOD-323, F.Cu at (288.8, 94.7)
- added D_R05_C16: 1N4148W, Arp3:D_SOD-323, F.Cu at (307.8, 94.7)
- added D_R06_C01: 1N4148W, Arp3:D_SOD-323, F.Cu at (22.1, 113.8)
- added D_R06_C02: 1N4148W, Arp3:D_SOD-323, F.Cu at (41.1, 113.8)
- added D_R06_C03: 1N4148W, Arp3:D_SOD-323, F.Cu at (60.2, 113.8)
- added D_R06_C04: 1N4148W, Arp3:D_SOD-323, F.Cu at (79.2, 113.8)
- added D_R06_C05: 1N4148W, Arp3:D_SOD-323, F.Cu at (98.3, 113.8)
- added D_R06_C06: 1N4148W, Arp3:D_SOD-323, F.Cu at (117.3, 113.8)
- added D_R06_C07: 1N4148W, Arp3:D_SOD-323, F.Cu at (136.4, 113.8)
- added D_R06_C08: 1N4148W, Arp3:D_SOD-323, F.Cu at (155.4, 113.8)
- added D_R06_C09: 1N4148W, Arp3:D_SOD-323, F.Cu at (174.5, 113.8)
- added D_R06_C10: 1N4148W, Arp3:D_SOD-323, F.Cu at (193.5, 113.8)
- added D_R06_C11: 1N4148W, Arp3:D_SOD-323, F.Cu at (212.6, 113.8)
- added D_R06_C12: 1N4148W, Arp3:D_SOD-323, F.Cu at (231.6, 113.8)
- added D_R06_C13: 1N4148W, Arp3:D_SOD-323, F.Cu at (250.7, 113.8)
- added D_R06_C14: 1N4148W, Arp3:D_SOD-323, F.Cu at (269.7, 113.8)
- added D_R06_C15: 1N4148W, Arp3:D_SOD-323, F.Cu at (288.8, 113.8)
- added D_R06_C16: 1N4148W, Arp3:D_SOD-323, F.Cu at (307.8, 113.8)
- added D_R07_C01: 1N4148W, Arp3:D_SOD-323, F.Cu at (22.1, 132.8)
- added D_R07_C02: 1N4148W, Arp3:D_SOD-323, F.Cu at (41.1, 132.8)
- added D_R07_C03: 1N4148W, Arp3:D_SOD-323, F.Cu at (60.2, 132.8)
- added D_R07_C04: 1N4148W, Arp3:D_SOD-323, F.Cu at (79.2, 132.8)
- added D_R07_C05: 1N4148W, Arp3:D_SOD-323, F.Cu at (98.3, 132.8)
- added D_R07_C06: 1N4148W, Arp3:D_SOD-323, F.Cu at (117.3, 132.8)
- added D_R07_C07: 1N4148W, Arp3:D_SOD-323, F.Cu at (136.4, 132.8)
- added D_R07_C08: 1N4148W, Arp3:D_SOD-323, F.Cu at (155.4, 132.8)
- added D_R07_C09: 1N4148W, Arp3:D_SOD-323, F.Cu at (174.5, 132.8)
- added D_R07_C10: 1N4148W, Arp3:D_SOD-323, F.Cu at (193.5, 132.8)
- added D_R07_C11: 1N4148W, Arp3:D_SOD-323, F.Cu at (212.6, 132.8)
- added D_R07_C12: 1N4148W, Arp3:D_SOD-323, F.Cu at (231.6, 132.8)
- added D_R07_C13: 1N4148W, Arp3:D_SOD-323, F.Cu at (250.7, 132.8)
- added D_R07_C14: 1N4148W, Arp3:D_SOD-323, F.Cu at (269.7, 132.8)
- added D_R07_C15: 1N4148W, Arp3:D_SOD-323, F.Cu at (288.8, 132.8)
- added D_R07_C16: 1N4148W, Arp3:D_SOD-323, F.Cu at (307.8, 132.8)
- added D_R08_C01: 1N4148W, Arp3:D_SOD-323, F.Cu at (22.1, 151.9)
- added D_R08_C02: 1N4148W, Arp3:D_SOD-323, F.Cu at (41.1, 151.9)
- added D_R08_C03: 1N4148W, Arp3:D_SOD-323, F.Cu at (60.2, 151.9)
- added D_R08_C04: 1N4148W, Arp3:D_SOD-323, F.Cu at (79.2, 151.9)
- added D_R08_C05: 1N4148W, Arp3:D_SOD-323, F.Cu at (98.3, 151.9)
- added D_R08_C06: 1N4148W, Arp3:D_SOD-323, F.Cu at (117.3, 151.9)
- added D_R08_C07: 1N4148W, Arp3:D_SOD-323, F.Cu at (136.4, 151.9)
- added D_R08_C08: 1N4148W, Arp3:D_SOD-323, F.Cu at (155.4, 151.9)
- added D_R08_C09: 1N4148W, Arp3:D_SOD-323, F.Cu at (174.5, 151.9)
- added D_R08_C10: 1N4148W, Arp3:D_SOD-323, F.Cu at (193.5, 151.9)
- added D_R08_C11: 1N4148W, Arp3:D_SOD-323, F.Cu at (212.6, 151.9)
- added D_R08_C12: 1N4148W, Arp3:D_SOD-323, F.Cu at (231.6, 151.9)
- added D_R08_C13: 1N4148W, Arp3:D_SOD-323, F.Cu at (250.7, 151.9)
- added D_R08_C14: 1N4148W, Arp3:D_SOD-323, F.Cu at (269.7, 151.9)
- added D_R08_C15: 1N4148W, Arp3:D_SOD-323, F.Cu at (288.8, 151.9)
- added D_R08_C16: 1N4148W, Arp3:D_SOD-323, F.Cu at (307.8, 151.9)
- added D_R09_C01: , Arp3:D_SOD-323, F.Cu at (3.02, 170.9)
- added D_R09_C02: , Arp3:D_SOD-323, F.Cu at (22.1, 170.9)
- added D_R09_C03: , Arp3:D_SOD-323, F.Cu at (41.1, 170.9)
- added D_R09_C04: , Arp3:D_SOD-323, F.Cu at (60.2, 170.9)
- added D_R09_C05: , Arp3:D_SOD-323, F.Cu at (79.2, 170.9)
- added D_R09_C06: , Arp3:D_SOD-323, F.Cu at (98.3, 170.9)
- added D_R09_C07: , Arp3:D_SOD-323, F.Cu at (117.3, 170.9)
- added D_R09_C08: , Arp3:D_SOD-323, F.Cu at (136.4, 170.9)
- added D_R09_C09: , Arp3:D_SOD-323, F.Cu at (155.4, 170.9)
- added J4: USB D+/D-, Arp3:USB_Dev_Pads, F.Cu at (381.9, 19.0)
- added LED_R01_C01: SK6812MINI-E, Arp3:SK6812MINI-E, F.Cu at (30.6, 6.83)
- added LED_R01_C02: SK6812MINI-E, Arp3:SK6812MINI-E, F.Cu at (49.6, 6.83)
- added LED_R01_C03: SK6812MINI-E, Arp3:SK6812MINI-E, F.Cu at (68.7, 6.83)
- added LED_R01_C04: SK6812MINI-E, Arp3:SK6812MINI-E, F.Cu at (87.7, 6.83)
- added LED_R01_C05: SK6812MINI-E, Arp3:SK6812MINI-E, F.Cu at (106.8, 6.83)
- added LED_R01_C06: SK6812MINI-E, Arp3:SK6812MINI-E, F.Cu at (125.8, 6.83)
- added LED_R01_C07: SK6812MINI-E, Arp3:SK6812MINI-E, F.Cu at (144.9, 6.83)
- added LED_R01_C08: SK6812MINI-E, Arp3:SK6812MINI-E, F.Cu at (163.9, 6.83)
- added LED_R01_C09: SK6812MINI-E, Arp3:SK6812MINI-E, F.Cu at (183.0, 6.83)
- added LED_R01_C10: SK6812MINI-E, Arp3:SK6812MINI-E, F.Cu at (202.0, 6.83)
- added LED_R01_C11: SK6812MINI-E, Arp3:SK6812MINI-E, F.Cu at (221.1, 6.83)
- added LED_R01_C12: SK6812MINI-E, Arp3:SK6812MINI-E, F.Cu at (240.1, 6.83)
- added LED_R01_C13: SK6812MINI-E, Arp3:SK6812MINI-E, F.Cu at (259.2, 6.83)
- added LED_R01_C14: SK6812MINI-E, Arp3:SK6812MINI-E, F.Cu at (278.2, 6.83)
- added LED_R01_C15: SK6812MINI-E, Arp3:SK6812MINI-E, F.Cu at (297.3, 6.83)
- added LED_R01_C16: SK6812MINI-E, Arp3:SK6812MINI-E, F.Cu at (316.3, 6.83)
- added LED_R02_C01: SK6812MINI-E, Arp3:SK6812MINI-E, F.Cu at (30.6, 25.9)
- added LED_R02_C02: SK6812MINI-E, Arp3:SK6812MINI-E, F.Cu at (49.6, 25.9)
- added LED_R02_C03: SK6812MINI-E, Arp3:SK6812MINI-E, F.Cu at (68.7, 25.9)
- added LED_R02_C04: SK6812MINI-E, Arp3:SK6812MINI-E, F.Cu at (87.7, 25.9)
- added LED_R02_C05: SK6812MINI-E, Arp3:SK6812MINI-E, F.Cu at (106.8, 25.9)
- added LED_R02_C06: SK6812MINI-E, Arp3:SK6812MINI-E, F.Cu at (125.8, 25.9)
- added LED_R02_C07: SK6812MINI-E, Arp3:SK6812MINI-E, F.Cu at (144.9, 25.9)
- added LED_R02_C08: SK6812MINI-E, Arp3:SK6812MINI-E, F.Cu at (163.9, 25.9)
- added LED_R02_C09: SK6812MINI-E, Arp3:SK6812MINI-E, F.Cu at (183.0, 25.9)
- added LED_R02_C10: SK6812MINI-E, Arp3:SK6812MINI-E, F.Cu at (202.0, 25.9)
- added LED_R02_C11: SK6812MINI-E, Arp3:SK6812MINI-E, F.Cu at (221.1, 25.9)
- added LED_R02_C12: SK6812MINI-E, Arp3:SK6812MINI-E, F.Cu at (240.1, 25.9)
- added LED_R02_C13: SK6812MINI-E, Arp3:SK6812MINI-E, F.Cu at (259.2, 25.9)
- added LED_R02_C14: SK6812MINI-E, Arp3:SK6812MINI-E, F.Cu at (278.2, 25.9)
- added LED_R02_C15: SK6812MINI-E, Arp3:SK6812MINI-E, F.Cu at (297.3, 25.9)
- added LED_R02_C16: SK6812MINI-E, Arp3:SK6812MINI-E, F.Cu at (316.3, 25.9)
- added LED_R03_C01: SK6812MINI-E, Arp3:SK6812MINI-E, F.Cu at (30.6, 44.9)
- added LED_R03_C02: SK6812MINI-E, Arp3:SK6812MINI-E, F.Cu at (49.6, 44.9)
- added LED_R03_C03: SK6812MINI-E, Arp3:SK6812MINI-E, F.Cu at (68.7, 44.9)
- added LED_R03_C04: SK6812MINI-E, Arp3:SK6812MINI-E, F.Cu at (87.7, 44.9)
- added LED_R03_C05: SK6812MINI-E, Arp3:SK6812MINI-E, F.Cu at (106.8, 44.9)
- added LED_R03_C06: SK6812MINI-E, Arp3:SK6812MINI-E, F.Cu at (125.8, 44.9)
- added LED_R03_C07: SK6812MINI-E, Arp3:SK6812MINI-E, F.Cu at (144.9, 44.9)
- added LED_R03_C08: SK6812MINI-E, Arp3:SK6812MINI-E, F.Cu at (163.9, 44.9)
- added LED_R03_C09: SK6812MINI-E, Arp3:SK6812MINI-E, F.Cu at (183.0, 44.9)
- added LED_R03_C10: SK6812MINI-E, Arp3:SK6812MINI-E, F.Cu at (202.0, 44.9)
- added LED_R03_C11: SK6812MINI-E, Arp3:SK6812MINI-E, F.Cu at (221.1, 44.9)
- added LED_R03_C12: SK6812MINI-E, Arp3:SK6812MINI-E, F.Cu at (240.1, 44.9)
- added LED_R03_C13: SK6812MINI-E, Arp3:SK6812MINI-E, F.Cu at (259.2, 44.9)
- added LED_R03_C14: SK6812MINI-E, Arp3:SK6812MINI-E, F.Cu at (278.2, 44.9)
- added LED_R03_C15: SK6812MINI-E, Arp3:SK6812MINI-E, F.Cu at (297.3, 44.9)
- added LED_R03_C16: SK6812MINI-E, Arp3:SK6812MINI-E, F.Cu at (316.3, 44.9)
- added LED_R04_C01: SK6812MINI-E, Arp3:SK6812MINI-E, F.Cu at (30.6, 64.0)
- added LED_R04_C02: SK6812MINI-E, Arp3:SK6812MINI-E, F.Cu at (49.6, 64.0)
- added LED_R04_C03: SK6812MINI-E, Arp3:SK6812MINI-E, F.Cu at (68.7, 64.0)
- added LED_R04_C04: SK6812MINI-E, Arp3:SK6812MINI-E, F.Cu at (87.7, 64.0)
- added LED_R04_C05: SK6812MINI-E, Arp3:SK6812MINI-E, F.Cu at (106.8, 64.0)
- added LED_R04_C06: SK6812MINI-E, Arp3:SK6812MINI-E, F.Cu at (125.8, 64.0)
- added LED_R04_C07: SK6812MINI-E, Arp3:SK6812MINI-E, F.Cu at (144.9, 64.0)
- added LED_R04_C08: SK6812MINI-E, Arp3:SK6812MINI-E, F.Cu at (163.9, 64.0)
- added LED_R04_C09: SK6812MINI-E, Arp3:SK6812MINI-E, F.Cu at (183.0, 64.0)
- added LED_R04_C10: SK6812MINI-E, Arp3:SK6812MINI-E, F.Cu at (202.0, 64.0)
- added LED_R04_C11: SK6812MINI-E, Arp3:SK6812MINI-E, F.Cu at (221.1, 64.0)
- added LED_R04_C12: SK6812MINI-E, Arp3:SK6812MINI-E, F.Cu at (240.1, 64.0)
- added LED_R04_C13: SK6812MINI-E, Arp3:SK6812MINI-E, F.Cu at (259.2, 64.0)
- added LED_R04_C14: SK6812MINI-E, Arp3:SK6812MINI-E, F.Cu at (278.2, 64.0)
- added LED_R04_C15: SK6812MINI-E, Arp3:SK6812MINI-E, F.Cu at (297.3, 64.0)
- added LED_R04_C16: SK6812MINI-E, Arp3:SK6812MINI-E, F.Cu at (316.3, 64.0)
- added LED_R05_C01: SK6812MINI-E, Arp3:SK6812MINI-E, F.Cu at (30.6, 83.0)
- added LED_R05_C02: SK6812MINI-E, Arp3:SK6812MINI-E, F.Cu at (49.6, 83.0)
- added LED_R05_C03: SK6812MINI-E, Arp3:SK6812MINI-E, F.Cu at (68.7, 83.0)
- added LED_R05_C04: SK6812MINI-E, Arp3:SK6812MINI-E, F.Cu at (87.7, 83.0)
- added LED_R05_C05: SK6812MINI-E, Arp3:SK6812MINI-E, F.Cu at (106.8, 83.0)
- added LED_R05_C06: SK6812MINI-E, Arp3:SK6812MINI-E, F.Cu at (125.8, 83.0)
- added LED_R05_C07: SK6812MINI-E, Arp3:SK6812MINI-E, F.Cu at (144.9, 83.0)
- added LED_R05_C08: SK6812MINI-E, Arp3:SK6812MINI-E, F.Cu at (163.9, 83.0)
- added LED_R05_C09: SK6812MINI-E, Arp3:SK6812MINI-E, F.Cu at (183.0, 83.0)
- added LED_R05_C10: SK6812MINI-E, Arp3:SK6812MINI-E, F.Cu at (202.0, 83.0)
- added LED_R05_C11: SK6812MINI-E, Arp3:SK6812MINI-E, F.Cu at (221.1, 83.0)
- added LED_R05_C12: SK6812MINI-E, Arp3:SK6812MINI-E, F.Cu at (240.1, 83.0)
- added LED_R05_C13: SK6812MINI-E, Arp3:SK6812MINI-E, F.Cu at (259.2, 83.0)
- added LED_R05_C14: SK6812MINI-E, Arp3:SK6812MINI-E, F.Cu at (278.2, 83.0)
- added LED_R05_C15: SK6812MINI-E, Arp3:SK6812MINI-E, F.Cu at (297.3, 83.0)
- added LED_R05_C16: SK6812MINI-E, Arp3:SK6812MINI-E, F.Cu at (316.3, 83.0)
- added LED_R06_C01: SK6812MINI-E, Arp3:SK6812MINI-E, F.Cu at (30.6, 102.1)
- added LED_R06_C02: SK6812MINI-E, Arp3:SK6812MINI-E, F.Cu at (49.6, 102.1)
- added LED_R06_C03: SK6812MINI-E, Arp3:SK6812MINI-E, F.Cu at (68.7, 102.1)
- added LED_R06_C04: SK6812MINI-E, Arp3:SK6812MINI-E, F.Cu at (87.7, 102.1)
- added LED_R06_C05: SK6812MINI-E, Arp3:SK6812MINI-E, F.Cu at (106.8, 102.1)
- added LED_R06_C06: SK6812MINI-E, Arp3:SK6812MINI-E, F.Cu at (125.8, 102.1)
- added LED_R06_C07: SK6812MINI-E, Arp3:SK6812MINI-E, F.Cu at (144.9, 102.1)
- added LED_R06_C08: SK6812MINI-E, Arp3:SK6812MINI-E, F.Cu at (163.9, 102.1)
- added LED_R06_C09: SK6812MINI-E, Arp3:SK6812MINI-E, F.Cu at (183.0, 102.1)
- added LED_R06_C10: SK6812MINI-E, Arp3:SK6812MINI-E, F.Cu at (202.0, 102.1)
- added LED_R06_C11: SK6812MINI-E, Arp3:SK6812MINI-E, F.Cu at (221.1, 102.1)
- added LED_R06_C12: SK6812MINI-E, Arp3:SK6812MINI-E, F.Cu at (240.1, 102.1)
- added LED_R06_C13: SK6812MINI-E, Arp3:SK6812MINI-E, F.Cu at (259.2, 102.1)
- added LED_R06_C14: SK6812MINI-E, Arp3:SK6812MINI-E, F.Cu at (278.2, 102.1)
- added LED_R06_C15: SK6812MINI-E, Arp3:SK6812MINI-E, F.Cu at (297.3, 102.1)
- added LED_R06_C16: SK6812MINI-E, Arp3:SK6812MINI-E, F.Cu at (316.3, 102.1)
- added LED_R07_C01: SK6812MINI-E, Arp3:SK6812MINI-E, F.Cu at (30.6, 121.1)
- added LED_R07_C02: SK6812MINI-E, Arp3:SK6812MINI-E, F.Cu at (49.6, 121.1)
- added LED_R07_C03: SK6812MINI-E, Arp3:SK6812MINI-E, F.Cu at (68.7, 121.1)
- added LED_R07_C04: SK6812MINI-E, Arp3:SK6812MINI-E, F.Cu at (87.7, 121.1)
- added LED_R07_C05: SK6812MINI-E, Arp3:SK6812MINI-E, F.Cu at (106.8, 121.1)
- added LED_R07_C06: SK6812MINI-E, Arp3:SK6812MINI-E, F.Cu at (125.8, 121.1)
- added LED_R07_C07: SK6812MINI-E, Arp3:SK6812MINI-E, F.Cu at (144.9, 121.1)
- added LED_R07_C08: SK6812MINI-E, Arp3:SK6812MINI-E, F.Cu at (163.9, 121.1)
- added LED_R07_C09: SK6812MINI-E, Arp3:SK6812MINI-E, F.Cu at (183.0, 121.1)
- added LED_R07_C10: SK6812MINI-E, Arp3:SK6812MINI-E, F.Cu at (202.0, 121.1)
- added LED_R07_C11: SK6812MINI-E, Arp3:SK6812MINI-E, F.Cu at (221.1, 121.1)
- added LED_R07_C12: SK6812MINI-E, Arp3:SK6812MINI-E, F.Cu at (240.1, 121.1)
- added LED_R07_C13: SK6812MINI-E, Arp3:SK6812MINI-E, F.Cu at (259.2, 121.1)
- added LED_R07_C14: SK6812MINI-E, Arp3:SK6812MINI-E, F.Cu at (278.2, 121.1)
- added LED_R07_C15: SK6812MINI-E, Arp3:SK6812MINI-E, F.Cu at (297.3, 121.1)
- added LED_R07_C16: SK6812MINI-E, Arp3:SK6812MINI-E, F.Cu at (316.3, 121.1)
- added LED_R08_C01: SK6812MINI-E, Arp3:SK6812MINI-E, F.Cu at (30.6, 140.2)
- added LED_R08_C02: SK6812MINI-E, Arp3:SK6812MINI-E, F.Cu at (49.6, 140.2)
- added LED_R08_C03: SK6812MINI-E, Arp3:SK6812MINI-E, F.Cu at (68.7, 140.2)
- added LED_R08_C04: SK6812MINI-E, Arp3:SK6812MINI-E, F.Cu at (87.7, 140.2)
- added LED_R08_C05: SK6812MINI-E, Arp3:SK6812MINI-E, F.Cu at (106.8, 140.2)
- added LED_R08_C06: SK6812MINI-E, Arp3:SK6812MINI-E, F.Cu at (125.8, 140.2)
- added LED_R08_C07: SK6812MINI-E, Arp3:SK6812MINI-E, F.Cu at (144.9, 140.2)
- added LED_R08_C08: SK6812MINI-E, Arp3:SK6812MINI-E, F.Cu at (163.9, 140.2)
- added LED_R08_C09: SK6812MINI-E, Arp3:SK6812MINI-E, F.Cu at (183.0, 140.2)
- added LED_R08_C10: SK6812MINI-E, Arp3:SK6812MINI-E, F.Cu at (202.0, 140.2)
- added LED_R08_C11: SK6812MINI-E, Arp3:SK6812MINI-E, F.Cu at (221.1, 140.2)
- added LED_R08_C12: SK6812MINI-E, Arp3:SK6812MINI-E, F.Cu at (240.1, 140.2)
- added LED_R08_C13: SK6812MINI-E, Arp3:SK6812MINI-E, F.Cu at (259.2, 140.2)
- added LED_R08_C14: SK6812MINI-E, Arp3:SK6812MINI-E, F.Cu at (278.2, 140.2)
- added LED_R08_C15: SK6812MINI-E, Arp3:SK6812MINI-E, F.Cu at (297.3, 140.2)
- added LED_R08_C16: SK6812MINI-E, Arp3:SK6812MINI-E, F.Cu at (316.3, 140.2)
- added SW_R01_C01: PG1350, Arp3:Kailh_Choc_V1, F.Cu at (30.6, 11.5)
- added SW_R01_C02: PG1350, Arp3:Kailh_Choc_V1, F.Cu at (49.6, 11.5)
- added SW_R01_C03: PG1350, Arp3:Kailh_Choc_V1, F.Cu at (68.7, 11.5)
- added SW_R01_C04: PG1350, Arp3:Kailh_Choc_V1, F.Cu at (87.7, 11.5)
- added SW_R01_C05: PG1350, Arp3:Kailh_Choc_V1, F.Cu at (106.8, 11.5)
- added SW_R01_C06: PG1350, Arp3:Kailh_Choc_V1, F.Cu at (125.8, 11.5)
- added SW_R01_C07: PG1350, Arp3:Kailh_Choc_V1, F.Cu at (144.9, 11.5)
- added SW_R01_C08: PG1350, Arp3:Kailh_Choc_V1, F.Cu at (163.9, 11.5)
- added SW_R01_C09: PG1350, Arp3:Kailh_Choc_V1, F.Cu at (183.0, 11.5)
- added SW_R01_C10: PG1350, Arp3:Kailh_Choc_V1, F.Cu at (202.0, 11.5)
- added SW_R01_C11: PG1350, Arp3:Kailh_Choc_V1, F.Cu at (221.1, 11.5)
- added SW_R01_C12: PG1350, Arp3:Kailh_Choc_V1, F.Cu at (240.1, 11.5)
- added SW_R01_C13: PG1350, Arp3:Kailh_Choc_V1, F.Cu at (259.2, 11.5)
- added SW_R01_C14: PG1350, Arp3:Kailh_Choc_V1, F.Cu at (278.2, 11.5)
- added SW_R01_C15: PG1350, Arp3:Kailh_Choc_V1, F.Cu at (297.3, 11.5)
- added SW_R01_C16: PG1350, Arp3:Kailh_Choc_V1, F.Cu at (316.3, 11.5)
- added SW_R02_C01: PG1350, Arp3:Kailh_Choc_V1, F.Cu at (30.6, 30.6)
- added SW_R02_C02: PG1350, Arp3:Kailh_Choc_V1, F.Cu at (49.6, 30.6)
- added SW_R02_C03: PG1350, Arp3:Kailh_Choc_V1, F.Cu at (68.7, 30.6)
- added SW_R02_C04: PG1350, Arp3:Kailh_Choc_V1, F.Cu at (87.7, 30.6)
- added SW_R02_C05: PG1350, Arp3:Kailh_Choc_V1, F.Cu at (106.8, 30.6)
- added SW_R02_C06: PG1350, Arp3:Kailh_Choc_V1, F.Cu at (125.8, 30.6)
- added SW_R02_C07: PG1350, Arp3:Kailh_Choc_V1, F.Cu at (144.9, 30.6)
- added SW_R02_C08: PG1350, Arp3:Kailh_Choc_V1, F.Cu at (163.9, 30.6)
- added SW_R02_C09: PG1350, Arp3:Kailh_Choc_V1, F.Cu at (183.0, 30.6)
- added SW_R02_C10: PG1350, Arp3:Kailh_Choc_V1, F.Cu at (202.0, 30.6)
- added SW_R02_C11: PG1350, Arp3:Kailh_Choc_V1, F.Cu at (221.1, 30.6)
- added SW_R02_C12: PG1350, Arp3:Kailh_Choc_V1, F.Cu at (240.1, 30.6)
- added SW_R02_C13: PG1350, Arp3:Kailh_Choc_V1, F.Cu at (259.2, 30.6)
- added SW_R02_C14: PG1350, Arp3:Kailh_Choc_V1, F.Cu at (278.2, 30.6)
- added SW_R02_C15: PG1350, Arp3:Kailh_Choc_V1, F.Cu at (297.3, 30.6)
- added SW_R02_C16: PG1350, Arp3:Kailh_Choc_V1, F.Cu at (316.3, 30.6)
- added SW_R03_C01: PG1350, Arp3:Kailh_Choc_V1, F.Cu at (30.6, 49.6)
- added SW_R03_C02: PG1350, Arp3:Kailh_Choc_V1, F.Cu at (49.6, 49.6)
- added SW_R03_C03: PG1350, Arp3:Kailh_Choc_V1, F.Cu at (68.7, 49.6)
- added SW_R03_C04: PG1350, Arp3:Kailh_Choc_V1, F.Cu at (87.7, 49.6)
- added SW_R03_C05: PG1350, Arp3:Kailh_Choc_V1, F.Cu at (106.8, 49.6)
- added SW_R03_C06: PG1350, Arp3:Kailh_Choc_V1, F.Cu at (125.8, 49.6)
- added SW_R03_C07: PG1350, Arp3:Kailh_Choc_V1, F.Cu at (144.9, 49.6)
- added SW_R03_C08: PG1350, Arp3:Kailh_Choc_V1, F.Cu at (163.9, 49.6)
- added SW_R03_C09: PG1350, Arp3:Kailh_Choc_V1, F.Cu at (183.0, 49.6)
- added SW_R03_C10: PG1350, Arp3:Kailh_Choc_V1, F.Cu at (202.0, 49.6)
- added SW_R03_C11: PG1350, Arp3:Kailh_Choc_V1, F.Cu at (221.1, 49.6)
- added SW_R03_C12: PG1350, Arp3:Kailh_Choc_V1, F.Cu at (240.1, 49.6)
- added SW_R03_C13: PG1350, Arp3:Kailh_Choc_V1, F.Cu at (259.2, 49.6)
- added SW_R03_C14: PG1350, Arp3:Kailh_Choc_V1, F.Cu at (278.2, 49.6)
- added SW_R03_C15: PG1350, Arp3:Kailh_Choc_V1, F.Cu at (297.3, 49.6)
- added SW_R03_C16: PG1350, Arp3:Kailh_Choc_V1, F.Cu at (316.3, 49.6)
- added SW_R04_C01: PG1350, Arp3:Kailh_Choc_V1, F.Cu at (30.6, 68.7)
- added SW_R04_C02: PG1350, Arp3:Kailh_Choc_V1, F.Cu at (49.6, 68.7)
- added SW_R04_C03: PG1350, Arp3:Kailh_Choc_V1, F.Cu at (68.7, 68.7)
- added SW_R04_C04: PG1350, Arp3:Kailh_Choc_V1, F.Cu at (87.7, 68.7)
- added SW_R04_C05: PG1350, Arp3:Kailh_Choc_V1, F.Cu at (106.8, 68.7)
- added SW_R04_C06: PG1350, Arp3:Kailh_Choc_V1, F.Cu at (125.8, 68.7)
- added SW_R04_C07: PG1350, Arp3:Kailh_Choc_V1, F.Cu at (144.9, 68.7)
- added SW_R04_C08: PG1350, Arp3:Kailh_Choc_V1, F.Cu at (163.9, 68.7)
- added SW_R04_C09: PG1350, Arp3:Kailh_Choc_V1, F.Cu at (183.0, 68.7)
- added SW_R04_C10: PG1350, Arp3:Kailh_Choc_V1, F.Cu at (202.0, 68.7)
- added SW_R04_C11: PG1350, Arp3:Kailh_Choc_V1, F.Cu at (221.1, 68.7)
- added SW_R04_C12: PG1350, Arp3:Kailh_Choc_V1, F.Cu at (240.1, 68.7)
- added SW_R04_C13: PG1350, Arp3:Kailh_Choc_V1, F.Cu at (259.2, 68.7)
- added SW_R04_C14: PG1350, Arp3:Kailh_Choc_V1, F.Cu at (278.2, 68.7)
- added SW_R04_C15: PG1350, Arp3:Kailh_Choc_V1, F.Cu at (297.3, 68.7)
- added SW_R04_C16: PG1350, Arp3:Kailh_Choc_V1, F.Cu at (316.3, 68.7)
- added SW_R05_C01: PG1350, Arp3:Kailh_Choc_V1, F.Cu at (30.6, 87.7)
- added SW_R05_C02: PG1350, Arp3:Kailh_Choc_V1, F.Cu at (49.6, 87.7)
- added SW_R05_C03: PG1350, Arp3:Kailh_Choc_V1, F.Cu at (68.7, 87.7)
- added SW_R05_C04: PG1350, Arp3:Kailh_Choc_V1, F.Cu at (87.7, 87.7)
- added SW_R05_C05: PG1350, Arp3:Kailh_Choc_V1, F.Cu at (106.8, 87.7)
- added SW_R05_C06: PG1350, Arp3:Kailh_Choc_V1, F.Cu at (125.8, 87.7)
- added SW_R05_C07: PG1350, Arp3:Kailh_Choc_V1, F.Cu at (144.9, 87.7)
- added SW_R05_C08: PG1350, Arp3:Kailh_Choc_V1, F.Cu at (163.9, 87.7)
- added SW_R05_C09: PG1350, Arp3:Kailh_Choc_V1, F.Cu at (183.0, 87.7)
- added SW_R05_C10: PG1350, Arp3:Kailh_Choc_V1, F.Cu at (202.0, 87.7)
- added SW_R05_C11: PG1350, Arp3:Kailh_Choc_V1, F.Cu at (221.1, 87.7)
- added SW_R05_C12: PG1350, Arp3:Kailh_Choc_V1, F.Cu at (240.1, 87.7)
- added SW_R05_C13: PG1350, Arp3:Kailh_Choc_V1, F.Cu at (259.2, 87.7)
- added SW_R05_C14: PG1350, Arp3:Kailh_Choc_V1, F.Cu at (278.2, 87.7)
- added SW_R05_C15: PG1350, Arp3:Kailh_Choc_V1, F.Cu at (297.3, 87.7)
- added SW_R05_C16: PG1350, Arp3:Kailh_Choc_V1, F.Cu at (316.3, 87.7)
- added SW_R06_C01: PG1350, Arp3:Kailh_Choc_V1, F.Cu at (30.6, 106.8)
- added SW_R06_C02: PG1350, Arp3:Kailh_Choc_V1, F.Cu at (49.6, 106.8)
- added SW_R06_C03: PG1350, Arp3:Kailh_Choc_V1, F.Cu at (68.7, 106.8)
- added SW_R06_C04: PG1350, Arp3:Kailh_Choc_V1, F.Cu at (87.7, 106.8)
- added SW_R06_C05: PG1350, Arp3:Kailh_Choc_V1, F.Cu at (106.8, 106.8)
- added SW_R06_C06: PG1350, Arp3:Kailh_Choc_V1, F.Cu at (125.8, 106.8)
- added SW_R06_C07: PG1350, Arp3:Kailh_Choc_V1, F.Cu at (144.9, 106.8)
- added SW_R06_C08: PG1350, Arp3:Kailh_Choc_V1, F.Cu at (163.9, 106.8)
- added SW_R06_C09: PG1350, Arp3:Kailh_Choc_V1, F.Cu at (183.0, 106.8)
- added SW_R06_C10: PG1350, Arp3:Kailh_Choc_V1, F.Cu at (202.0, 106.8)
- added SW_R06_C11: PG1350, Arp3:Kailh_Choc_V1, F.Cu at (221.1, 106.8)
- added SW_R06_C12: PG1350, Arp3:Kailh_Choc_V1, F.Cu at (240.1, 106.8)
- added SW_R06_C13: PG1350, Arp3:Kailh_Choc_V1, F.Cu at (259.2, 106.8)
- added SW_R06_C14: PG1350, Arp3:Kailh_Choc_V1, F.Cu at (278.2, 106.8)
- added SW_R06_C15: PG1350, Arp3:Kailh_Choc_V1, F.Cu at (297.3, 106.8)
- added SW_R06_C16: PG1350, Arp3:Kailh_Choc_V1, F.Cu at (316.3, 106.8)
- added SW_R07_C01: PG1350, Arp3:Kailh_Choc_V1, F.Cu at (30.6, 125.8)
- added SW_R07_C02: PG1350, Arp3:Kailh_Choc_V1, F.Cu at (49.6, 125.8)
- added SW_R07_C03: PG1350, Arp3:Kailh_Choc_V1, F.Cu at (68.7, 125.8)
- added SW_R07_C04: PG1350, Arp3:Kailh_Choc_V1, F.Cu at (87.7, 125.8)
- added SW_R07_C05: PG1350, Arp3:Kailh_Choc_V1, F.Cu at (106.8, 125.8)
- added SW_R07_C06: PG1350, Arp3:Kailh_Choc_V1, F.Cu at (125.8, 125.8)
- added SW_R07_C07: PG1350, Arp3:Kailh_Choc_V1, F.Cu at (144.9, 125.8)
- added SW_R07_C08: PG1350, Arp3:Kailh_Choc_V1, F.Cu at (163.9, 125.8)
- added SW_R07_C09: PG1350, Arp3:Kailh_Choc_V1, F.Cu at (183.0, 125.8)
- added SW_R07_C10: PG1350, Arp3:Kailh_Choc_V1, F.Cu at (202.0, 125.8)
- added SW_R07_C11: PG1350, Arp3:Kailh_Choc_V1, F.Cu at (221.1, 125.8)
- added SW_R07_C12: PG1350, Arp3:Kailh_Choc_V1, F.Cu at (240.1, 125.8)
- added SW_R07_C13: PG1350, Arp3:Kailh_Choc_V1, F.Cu at (259.2, 125.8)
- added SW_R07_C14: PG1350, Arp3:Kailh_Choc_V1, F.Cu at (278.2, 125.8)
- added SW_R07_C15: PG1350, Arp3:Kailh_Choc_V1, F.Cu at (297.3, 125.8)
- added SW_R07_C16: PG1350, Arp3:Kailh_Choc_V1, F.Cu at (316.3, 125.8)
- added SW_R08_C01: PG1350, Arp3:Kailh_Choc_V1, F.Cu at (30.6, 144.9)
- added SW_R08_C02: PG1350, Arp3:Kailh_Choc_V1, F.Cu at (49.6, 144.9)
- added SW_R08_C03: PG1350, Arp3:Kailh_Choc_V1, F.Cu at (68.7, 144.9)
- added SW_R08_C04: PG1350, Arp3:Kailh_Choc_V1, F.Cu at (87.7, 144.9)
- added SW_R08_C05: PG1350, Arp3:Kailh_Choc_V1, F.Cu at (106.8, 144.9)
- added SW_R08_C06: PG1350, Arp3:Kailh_Choc_V1, F.Cu at (125.8, 144.9)
- added SW_R08_C07: PG1350, Arp3:Kailh_Choc_V1, F.Cu at (144.9, 144.9)
- added SW_R08_C08: PG1350, Arp3:Kailh_Choc_V1, F.Cu at (163.9, 144.9)
- added SW_R08_C09: PG1350, Arp3:Kailh_Choc_V1, F.Cu at (183.0, 144.9)
- added SW_R08_C10: PG1350, Arp3:Kailh_Choc_V1, F.Cu at (202.0, 144.9)
- added SW_R08_C11: PG1350, Arp3:Kailh_Choc_V1, F.Cu at (221.1, 144.9)
- added SW_R08_C12: PG1350, Arp3:Kailh_Choc_V1, F.Cu at (240.1, 144.9)
- added SW_R08_C13: PG1350, Arp3:Kailh_Choc_V1, F.Cu at (259.2, 144.9)
- added SW_R08_C14: PG1350, Arp3:Kailh_Choc_V1, F.Cu at (278.2, 144.9)
- added SW_R08_C15: PG1350, Arp3:Kailh_Choc_V1, F.Cu at (297.3, 144.9)
- added SW_R08_C16: PG1350, Arp3:Kailh_Choc_V1, F.Cu at (316.3, 144.9)
- added SW_R09_C01: , Arp3:Kailh_Choc_V1, F.Cu at (11.5, 163.9)
- added SW_R09_C02: , Arp3:Kailh_Choc_V1, F.Cu at (30.6, 163.9)
- added SW_R09_C03: , Arp3:Kailh_Choc_V1, F.Cu at (49.6, 163.9)
- added SW_R09_C04: , Arp3:Kailh_Choc_V1, F.Cu at (68.7, 163.9)
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Connections:
- C9 pad 1: VCC -> GND
- C9 pad 2: GND -> VCC
- U3 pad L10: (no net) -> DISP_LED
- U3 pad L12: (no net) -> DISP_CS
- U3 pad L13: (no net) -> DISP_MOSI
- U3 pad L14: (no net) -> DISP_MISO
- U3 pad L8: (no net) -> DISP_DC
- U3 pad L9: (no net) -> DISP_RST
- U3 pad R14: (no net) -> DISP_SCK
Routing:
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- added copper zone on F.Cu, net LED_VCC
- removed copper zone on B.Cu, net LED_VCC
- removed copper zone on F.Cu, net VCC
